File: hardware/kicad/HubAudio/HubAudio.kicad_sch (KiCad schematic)
At the start: 0 parts

Commit message: Update HubAudio hardware, schematics and architecture
Other:
- added sheet Antenna (antenna.kicad_sch)
- added sheet AudioDomainController (audiodomaincontroller.kicad_sch)
- added sheet AudioProcessor (audio-processor.kicad_sch)
- added sheet BT-Unit (BT-Unit.kicad_sch)
- added sheet Coder (Codec.kicad_sch)
- added sheet DeviceManager (device-manager.kicad_sch)
- added sheet Ethernet (ethernet.kicad_sch)
- added sheet Main Controller (main-controller.kicad_sch)
- added sheet POWER (POWER.kicad_sch)
- added sheet PowerDistribution (powerdistribution.kicad_sch)
- added sheet Si4684 (Si4684.kicad_sch)
- added sheet USB (USB.kicad_sch)

Commit message: Finalize I2C and SPI control architecture
Other:
- sheet AudioDomainController renamed PowerDistribution_2
- sheet Coder renamed Codec
- note added: ".global 0"
Changed lines of the file:
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@@
 	(generator_version "10.0")
 	(paper "A4")
+	(text ".global 0"
+		(exclude_from_sim no)
+		(at 58.42 139.954 0)
+		(effects
+			(font
+				(size 1.27 1.27)
+			)
+		)
+	)
 	(sheet
 		(at 85.09 25.4)
@@
 			(project "HubAudio"
 				(path "/841d8022-3a94-443e-97aa-a99a12889684"
-					(page "9")
+					(page "10")
 				)
 			)
@@
 			(project "HubAudio"
 				(path "/841d8022-3a94-443e-97aa-a99a12889684"
-					(page "11")
+					(page "12")
 				)
 			)
@@
 			(project "HubAudio"
 				(path "/841d8022-3a94-443e-97aa-a99a12889684"
-					(page "10")
+					(page "11")
 				)
 			)
@@
 			(project "HubAudio"
 				(path "/841d8022-3a94-443e-97aa-a99a12889684"
-					(page "4")
+					(page "6")
 				)
 			)
@@
 			(color 0 0 0 0)
 		)
-		(property "Sheetname" "AudioDomainController"
+		(property "Sheetname" "PowerDistribution_2"
 			(at 26.67 102.1584 0)
 			(show_name no)
@@
 			(project "HubAudio"
 				(path "/841d8022-3a94-443e-97aa-a99a12889684"
-					(page "12")
+					(page "4")
 				)
 			)
@@
 			(project "HubAudio"
 				(path "/841d8022-3a94-443e-97aa-a99a12889684"
-					(page "7")
+					(page "8")
 				)
 			)
@@
 			(color 0 0 0 0)
 		)
-		(property "Sheetname" "Coder"
+		(property "Sheetname" "Codec"
 			(at 85.09 65.3284 0)
 			(show_name no)
@@
 			(project "HubAudio"
 				(path "/841d8022-3a94-443e-97aa-a99a12889684"
-					(page "8")
+					(page "9")
 				)
 			)
@@
 			(project "HubAudio"
 				(path "/841d8022-3a94-443e-97aa-a99a12889684"
-					(page "6")
-				)
-			)
+					(page "7")
+				)
+			)
