File: hardware/kicad/HubAudio/audiodomaincontroller.kicad_sch (KiCad schematic)
At the start: 0 parts

Commit message: Finalize I2C and SPI control architecture
Parts:
- added C120, C153, C154, C155, C156, C157, C180, C181, C182, C183: 1uF, Capacitor_SMD:C_0805_2012Metric, symbol Device:C
- added C149, C150, C151, C152: 22uF, Capacitor_SMD:C_0805_2012Metric, symbol Device:C
- added C158, C175, C176, C177, C178, C179, C39, C42: 10uF, Capacitor_SMD:C_1206_3216Metric, symbol Device:C
- added C184, C185, C186, C187, C191, C192, C193, C194: 100nF, Capacitor_SMD:C_0805_2012Metric, symbol Device:C
- added L21, L22, L23, L24: ferrite bead, Inductor_SMD:L_0805_2012Metric, symbol Device:L
- added U23: TPS22994RUKT, MIKILAB_TPS22994RUKT:IC_TPS22994RUKT, symbol MIKILAB_TPS22994RUKT:TPS22994RUKT
- added U31, U32, U33, U37: TMP117NAIDRVR, Package_SON:WSON-6-1EP_2x2mm_P0.65mm_EP1x1.6mm, symbol MIKILAB_Sensor_Temperature:TMP117xxDRV
Connections:
- new net: C42.1, L22.1, U23.1 (VOUT2)
- new net: C158.1, L23.1, U23.15 (VOUT3)
- new net: C39.1, L21.1, U23.5 (VOUT1)
- new net: C175.1, L24.1, U23.11 (VOUT4)
- new net 1V8: C150.2, C152.2, C154.2, C156.1, U23.12 (VIN4), U23.2 (VIN2)
- new net 1V8_CODER: C177.1, C181.1, C185.1, L22.2
- new net 1V8_SI4684: C179.1, C183.1, C187.1, L24.2
- new net 3V3_ANALOG: C149.2, C151.2, C153.1, C155.1, U23.14 (VIN3), U23.4 (VIN1)
- new net 3V3_CODER: C176.1, C180.1, C184.1, L21.2
- new net 3V3_DIGITAL: C120.2, C157.2, C191.2, C192.2, C193.2, C194.2, U23.18 (VDD), U23.3 (VBIAS), U23.6 (ADD1), U31.5 (V+), U32.5 (V+), U33.4 (ADD0), U33.5 (V+), U37.5 (V+)
- new net 3V3_SI4684: C178.1, C182.1, C186.1, L23.2
- new net GND: C120.1, C149.1, C150.1, C151.1, C152.1, C153.2, C154.1, C155.2, C156.2, C157.1, C158.2, C175.2, C176.2, C177.2, C178.2, C179.2, C180.2, C181.2, C182.2, C183.2, C184.2, C185.2, C186.2, C187.2, C191.1, C192.1, C193.1, C194.1, C39.2, C42.2, U23.10 (ON1), U23.13 (GND), U23.16 (ADD2), U23.20 (ADD3), U23.21 (EXP), U23.7 (ON4), U23.8 (ON3), U23.9 (ON2), U31.2 (GND), U31.4 (ADD0), U32.2 (GND), U33.2 (GND), U37.2 (GND)
- new net I2C_SCL: U23.17 (SCL), U31.1 (SCL), U32.1 (SCL), U33.1 (SCL), U37.1 (SCL), U37.4 (ADD0)
- new net I2C_SDA: U23.19 (SDA), U31.6 (SDA), U32.4 (ADD0), U32.6 (SDA), U33.6 (SDA), U37.6 (SDA)
- new net TEMP_ALERT_CODEC: U37.3 (ALERT)
- new net TEMP_ALERT_DSP: U32.3 (ALERT)
- new net TEMP_ALERT_ESP32: U33.3 (ALERT)
- new net TEMP_ALERT_POWER: U31.3 (ALERT)
