File: hardware/kicad/HubAudio/Si4684.kicad_sch (KiCad schematic)
At the start: 21 parts, among them U12 Si4684-A10-GM, U29 SST25VF080B-50-4x-S2Ax, Y2 ABM8-19.200MHZ-10-1-U-T

Commit message: Finalize I2C and SPI control architecture
Parts:
- removed U29: SST25VF080B-50-4x-S2Ax, Package_SO:SOIC-8_5.275x5.275mm_P1.27mm, symbol MIKILAB_Memory_Flash:SST25VF080B-50-4x-S2Ax
- added R95: 33, Resistor_SMD:R_0805_2012Metric, symbol Device:R
- added U27: W25Q16JW, Package_SO:SOIC-8_5.23x5.23mm_P1.27mm, symbol MIKILAB_Memory_Flash:W25Q16JVSS
- C103, C106, C109, C112: PNM (none) -> GQM2195C2E8R2CB12D
- C104, C107, C110, C113: PNM (none) -> GRM2165C1H222JA01D
- C105, C108, C111, C114, C117: PNM (none) -> GCM21BR71E105KA56L
- C115, C116: PNM (none) -> GQM2195C2E150JB12D
- C119: PNM (none) -> GRM21BR71H104KA01L
- R58, R59: PNM (none) -> RC0805FR-0710KL
- U12: PNM (none) -> Si4684-A10-GM
Connections:
- net SI4684_RREF is gone; now on net GND: U12.6 (RFREF), U12.7 (RFREF), U12.8 (RFREF), U12.9 (RFREF)
- net 1V8_SI4684: now also U27.8 (VCC)
- net GND: now also U27.4 (GND)
- net I2S_IN_RADIO_BCLK: now also U12.27 (DCLK); no longer U12.3 (INTB)
- net I2S_IN_RADIO_LRCLK: now also U12.28 (DFS); no longer U12.27 (DCLK)
- net I2S_IN_RADIO_SDATA: now also R95.2; no longer U12.28 (DFS)
- net NV_CLK: now also U27.6 (CLK)
- net NV_MISO: now also U27.2 (DO(IO1))
- net NV_MOSI: now also U27.5 (DI(IO0))
- net NV_SSB: now also U27.1 (~{CS})
- net SI4684_INT: now also U12.3 (INTB); no longer U12.33 (DOUT)
- net at R58.1: now also U27.3 (IO2)
- net at R59.1: now also U27.7 (IO3)
- new net: R95.1, U12.33 (DOUT)
- no-connect marks 0 -> 2

Commit message: Finalize HubAudio hardware architecture and PCB
Parts:
- U27: footprint Package_SO:SOIC-8_5.23x5.23mm_P1.27mm -> Package_SO:SOIC-8_5.3x5.3mm_P1.27mm
Changed lines of the file:
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@@
 			)
 		)
-		(property "Footprint" "Package_SO:SOIC-8_5.23x5.23mm_P1.27mm"
+		(property "Footprint" "Package_SO:SOIC-8_5.3x5.3mm_P1.27mm"
 			(at 134.62 152.4 0)
 			(hide yes)
