File: hardware/kicad/HubAudio/audio-processor.kicad_sch (KiCad schematic)
At the start: 41 parts, among them J3 AFBR-1624Z, J4 AFBR-2529Z, U18 ADAU1467WBCPZ300R, U24 25AA1024-I_SM, Y1 ABM3B-12.288MHZ-10-1-U-T

Commit message: Finalize I2C and SPI control architecture
Parts:
- C29, C30: PNM (none) -> CL21C220JBANNNC
- C31, C32, C84, C85: PNM (none) -> GRM21BR61E106KA73L
- C33, C72, C73, C74, C75, C76, C77, C78, C79, C80, C86: PNM (none) -> GRM21BR71H104KA01L
- C70: value 100NF -> 100nF; PNM (none) -> GRM21BR71H104KA01L
- C81: PNM (none) -> 08055A151FAT2A
- C82: PNM (none) -> GCM2195C1K562FA16D
- L10, L5: value LSQNB160808T470M -> ferrite bead; PNM (none) -> LSQNB160808T470M
- R46: PNM (none) -> 0805W8F4301T5E; now left out of the parts list
- R47, R48: PNM (none) -> RC0805FR-0710KL
- R51: value 10K -> 100; PNM (none) -> RC0805FR-07100RL
- R52: PNM (none) -> RC0805FR-074K7L
- RN10, RN2, RN3, RN4, RN5, RN6, RN7, RN8, RN9: value 0 OHM -> 33; PNM (none) -> YC164-JR-0733RL; now left out of the parts list
- U18: PNM (none) -> ADAU1467WBCPZ300R
- U24: PNM (none) -> 25AA1024-I_SM
Connections:
- no-connect marks 0 -> 30

Commit message: Finalize HubAudio hardware architecture and PCB
Parts:
- added C88: 100nF, Capacitor_SMD:C_0805_2012Metric, symbol Device:C
Connections:
- net 3V3_ADAU1467: now also C88.2
- net GND: now also C88.1
- net I2S_IN_BT1058_SDATA: now reaches U18.86 (SDATA_IN3)
- net I2S_OUT_BT1035_BCLK renamed I2S_OUT_BT1058_BCLK
- net I2S_OUT_BT1035_LRCLK renamed I2S_OUT_BT1058_LRCLK
- net I2S_OUT_BT1035_SDATA renamed I2S_OUT_BT1058_SDATA
- no-connect marks 30 -> 29
