File: hardware/kicad/HubAudio/HubAudio.kicad_pcb (KiCad board)
At the start: 2 copper layers, 95 x 75 mm, 4 parts

Commit message: Update PCB power placement
Parts:
- added BOOT1: TS3425UA-3x4x2.5-160, MIKILAB_TS3425UA_3x4x2_5_160:TS3425UA-3x4x2.5-160, F.Cu at (-161.2, 98.2)
- added C1: 10uF, Capacitor_SMD:C_1206_3216Metric, B.Cu at (189.8, 71.5)
- added C10: 1uF, Capacitor_SMD:C_1206_3216Metric, B.Cu at (189.8, 84.8)
- added C100: 33pF, Capacitor_SMD:C_0603_1608Metric, F.Cu at (-103.5, 102.6)
- added C101: 2.7pF, Capacitor_SMD:C_0603_1608Metric, F.Cu at (-103.5, 105.1)
- added C102: 18pF, Capacitor_SMD:C_0805_2012Metric, F.Cu at (-101.4, 99.7)
- added C103: 8.2pF, Capacitor_SMD:C_0805_2012Metric, F.Cu at (-148.0, 155.2)
- added C104: 2.2nF, Capacitor_SMD:C_0805_2012Metric, F.Cu at (-148.0, 158.2)
- added C105: 1uF, Capacitor_SMD:C_0805_2012Metric, F.Cu at (-148.0, 161.2)
- added C106: 8.2pF, Capacitor_SMD:C_0805_2012Metric, F.Cu at (-148.0, 164.2)
- added C107: 2.2nF, Capacitor_SMD:C_0805_2012Metric, F.Cu at (-143.5, 155.2)
- added C108: 1uF, Capacitor_SMD:C_0805_2012Metric, F.Cu at (-143.5, 158.2)
- added C109: 8.2pF, Capacitor_SMD:C_0805_2012Metric, F.Cu at (-143.5, 161.2)
- added C11: 100nF, Capacitor_SMD:C_0805_2012Metric, B.Cu at (66.0, 114.5)
- added C110: 2.2nF, Capacitor_SMD:C_0805_2012Metric, F.Cu at (-143.5, 164.2)
- added C111: 1uF, Capacitor_SMD:C_0805_2012Metric, F.Cu at (-139.1, 155.2)
- added C112: 8.2pF, Capacitor_SMD:C_0805_2012Metric, F.Cu at (-139.1, 158.2)
- added C113: 2.2nF, Capacitor_SMD:C_0805_2012Metric, F.Cu at (-139.1, 161.2)
- added C114: 1uF, Capacitor_SMD:C_0805_2012Metric, F.Cu at (-139.1, 164.2)
- added C115: 15pF, Capacitor_SMD:C_0805_2012Metric, F.Cu at (-134.6, 155.2)
- added C116: 15pF, Capacitor_SMD:C_0805_2012Metric, F.Cu at (-134.6, 158.2)
- added C117: 1uF, Capacitor_SMD:C_0805_2012Metric, F.Cu at (-134.6, 161.2)
- added C118: 47uF, Capacitor_SMD:C_1206_3216Metric, B.Cu at (178.5, 81.5)
- added C119: 100nF, Capacitor_SMD:C_0805_2012Metric, F.Cu at (-134.6, 164.2)
- added C12: 22uF, Capacitor_SMD:C_1206_3216Metric, B.Cu at (68.5, 120.0)
- added C120: 1uF, Capacitor_SMD:C_0805_2012Metric, F.Cu at (-121.3, 124.1)
- added C121: 10uF, Capacitor_SMD:C_1206_3216Metric, F.Cu at (-136.1, 115.6)
- added C122: 10uF, Capacitor_SMD:C_1206_3216Metric, F.Cu at (-136.1, 118.9)
- added C123: 1uF, Capacitor_SMD:C_0805_2012Metric, F.Cu at (-139.1, 93.7)
- added C124: 100nF, Capacitor_SMD:C_0805_2012Metric, F.Cu at (-139.1, 96.7)
- added C129: 100nF, Capacitor_SMD:C_0805_2012Metric, F.Cu at (-132.4, 124.1)
- added C13: 22uF, Capacitor_SMD:C_1206_3216Metric, B.Cu at (66.0, 120.0)
- added C132: 20pF, Capacitor_SMD:C_0805_2012Metric, F.Cu at (-132.4, 127.1)
- added C133: 20pF, Capacitor_SMD:C_0805_2012Metric, F.Cu at (-132.4, 130.1)
- added C134: 100nF, Capacitor_SMD:C_0805_2012Metric, F.Cu at (-132.4, 133.1)
- added C135: 100nF, Capacitor_SMD:C_0805_2012Metric, F.Cu at (-132.4, 136.2)
- added C136: 10uF, Capacitor_SMD:C_0805_2012Metric, F.Cu at (-132.4, 139.2)
- added C14: 10uF, Capacitor_SMD:C_1206_3216Metric, F.Cu at (-147.4, 108.9)
- added C141: 1uF, Capacitor_SMD:C_0805_2012Metric, F.Cu at (-139.1, 99.7)
- added C142: 1uF, Capacitor_SMD:C_0805_2012Metric, F.Cu at (-139.1, 102.7)
- added C143: 1uF, Capacitor_SMD:C_0805_2012Metric, F.Cu at (-139.1, 105.7)
- added C144: 1uF, Capacitor_SMD:C_0805_2012Metric, F.Cu at (-134.6, 90.7)
- added C145: 22uF, Capacitor_SMD:C_0805_2012Metric, F.Cu at (-134.6, 93.7)
- added C146: 22uF, Capacitor_SMD:C_0805_2012Metric, F.Cu at (-134.6, 96.7)
- added C147: 22uF, Capacitor_SMD:C_0805_2012Metric, F.Cu at (-134.6, 99.7)
- added C148: 22uF, Capacitor_SMD:C_0805_2012Metric, F.Cu at (-134.6, 102.7)
- added C149: 22uF, Capacitor_SMD:C_0805_2012Metric, F.Cu at (-121.3, 127.1)
- added C15: 1uF, Capacitor_SMD:C_1206_3216Metric, F.Cu at (-147.4, 112.2)
- added C150: 22uF, Capacitor_SMD:C_0805_2012Metric, F.Cu at (-121.3, 130.1)
- added C151: 22uF, Capacitor_SMD:C_0805_2012Metric, F.Cu at (-121.3, 133.1)
- added C152: 22uF, Capacitor_SMD:C_0805_2012Metric, F.Cu at (-121.3, 136.2)
- added C153: 1uF, Capacitor_SMD:C_0805_2012Metric, F.Cu at (-121.3, 139.2)
- added C154: 1uF, Capacitor_SMD:C_0805_2012Metric, F.Cu at (-116.8, 124.1)
- added C155: 1uF, Capacitor_SMD:C_0805_2012Metric, F.Cu at (-116.8, 127.1)
- added C156: 1uF, Capacitor_SMD:C_0805_2012Metric, F.Cu at (-116.8, 130.1)
- added C157: 1uF, Capacitor_SMD:C_0805_2012Metric, F.Cu at (-116.8, 133.1)
- added C158: 10uF, Capacitor_SMD:C_1206_3216Metric, F.Cu at (-102.9, 131.0)
- added C159: 100nF, Capacitor_SMD:C_0805_2012Metric, F.Cu at (-162.2, 122.2)
- added C16: 100nF, Capacitor_SMD:C_0805_2012Metric, F.Cu at (-148.0, 90.7)
- added C160: 100nF, Capacitor_SMD:C_0805_2012Metric, F.Cu at (-94.7, 61.5)
- added C161: 100nF, Capacitor_SMD:C_0805_2012Metric, F.Cu at (-94.7, 64.5)
- added C162: 100nF, Capacitor_SMD:C_0805_2012Metric, F.Cu at (-168.1, 45.0)
- added C163: 100nF, Capacitor_SMD:C_0805_2012Metric, F.Cu at (-168.1, 48.0)
- added C164: 10uF, Capacitor_SMD:C_0805_2012Metric, F.Cu at (-168.1, 51.0)
- added C165: 1uF, Capacitor_SMD:C_0805_2012Metric, F.Cu at (-168.1, 54.0)
- added C166: 1uF, Capacitor_SMD:C_0805_2012Metric, F.Cu at (-163.7, 45.0)
- added C167: 1uF, Capacitor_SMD:C_0805_2012Metric, F.Cu at (-163.7, 48.0)
- added C168: 1uF, Capacitor_SMD:C_0805_2012Metric, F.Cu at (-163.7, 51.0)
- added C169: 1uF, Capacitor_SMD:C_0805_2012Metric, F.Cu at (-163.7, 54.0)
- added C17: 1uF, Capacitor_SMD:C_1206_3216Metric, B.Cu at (74.8, 109.6)
- added C170: 1uF, Capacitor_SMD:C_0805_2012Metric, F.Cu at (-159.2, 45.0)
- added C171: 1uF, Capacitor_SMD:C_0805_2012Metric, F.Cu at (-159.2, 48.0)
- added C172: 1uF, Capacitor_SMD:C_0805_2012Metric, F.Cu at (-159.2, 51.0)
- added C173: 1uF, Capacitor_SMD:C_0805_2012Metric, F.Cu at (-159.2, 54.0)
- added C174: 100nF, Capacitor_SMD:C_0805_2012Metric, F.Cu at (-154.8, 45.0)
- added C175: 10uF, Capacitor_SMD:C_1206_3216Metric, F.Cu at (-102.9, 134.3)
- added C176: 10uF, Capacitor_SMD:C_1206_3216Metric, F.Cu at (-102.9, 137.7)
- added C177: 10uF, Capacitor_SMD:C_1206_3216Metric, F.Cu at (-102.9, 141.0)
- added C178: 10uF, Capacitor_SMD:C_1206_3216Metric, F.Cu at (-102.9, 144.4)
- added C179: 10uF, Capacitor_SMD:C_1206_3216Metric, F.Cu at (-102.9, 147.7)
- added C18: 1uF, Capacitor_SMD:C_1206_3216Metric, B.Cu at (51.5, 113.0)
- added C180: 1uF, Capacitor_SMD:C_0805_2012Metric, F.Cu at (-116.8, 136.2)
- added C181: 1uF, Capacitor_SMD:C_0805_2012Metric, F.Cu at (-116.8, 139.2)
- added C182: 1uF, Capacitor_SMD:C_0805_2012Metric, F.Cu at (-112.4, 124.1)
- added C183: 1uF, Capacitor_SMD:C_0805_2012Metric, F.Cu at (-112.4, 127.1)
- added C184: 100nF, Capacitor_SMD:C_0805_2012Metric, F.Cu at (-112.4, 130.1)
- added C185: 100nF, Capacitor_SMD:C_0805_2012Metric, F.Cu at (-112.4, 133.1)
- added C186: 100nF, Capacitor_SMD:C_0805_2012Metric, F.Cu at (-112.4, 136.2)
- added C187: 100nF, Capacitor_SMD:C_0805_2012Metric, F.Cu at (-112.4, 139.2)
- added C188: 1uF, Capacitor_SMD:C_0805_2012Metric, F.Cu at (-154.8, 48.0)
- added C189: 100nF, Capacitor_SMD:C_0805_2012Metric, F.Cu at (-154.8, 51.0)
- added C19: 1uF, Capacitor_SMD:C_1206_3216Metric, B.Cu at (80.8, 109.6)
- added C190: 1uF, Capacitor_SMD:C_0805_2012Metric, F.Cu at (-154.8, 54.0)
- added C191: 100nF, Capacitor_SMD:C_0805_2012Metric, F.Cu at (-107.9, 124.1)
- added C192: 100nF, Capacitor_SMD:C_0805_2012Metric, F.Cu at (-107.9, 127.1)
- added C193: 100nF, Capacitor_SMD:C_0805_2012Metric, F.Cu at (-107.9, 130.1)
- added C194: 100nF, Capacitor_SMD:C_0805_2012Metric, F.Cu at (-107.9, 133.1)
- added C2: 10uF, Capacitor_SMD:C_1206_3216Metric, B.Cu at (189.8, 74.8)
- added C20: 1uF, Capacitor_SMD:C_1206_3216Metric, B.Cu at (57.5, 113.0)
- added C21: 100nF, Capacitor_SMD:C_0805_2012Metric, B.Cu at (194.8, 89.3)
- added C22: 100nF, Capacitor_SMD:C_0805_2012Metric, B.Cu at (194.8, 92.3)
- added C23: 47uF, Capacitor_SMD:C_1206_3216Metric, B.Cu at (178.5, 74.8)
- added C25: 10uF, Capacitor_SMD:C_1206_3216Metric, F.Cu at (-147.4, 115.6)
- added C26: 10uF, Capacitor_SMD:C_1206_3216Metric, F.Cu at (-147.4, 118.9)
- added C27: 1uF, Capacitor_SMD:C_0805_2012Metric, F.Cu at (-148.0, 93.7)
- added C28: 100nF, Capacitor_SMD:C_0805_2012Metric, F.Cu at (-148.0, 96.7)
- added C29: 22pF, Capacitor_SMD:C_0805_2012Metric, F.Cu at (-129.1, 45.0)
- added C3: 100nF, Capacitor_SMD:C_0805_2012Metric, B.Cu at (194.8, 71.3)
- added C30: 22pF, Capacitor_SMD:C_0805_2012Metric, F.Cu at (-129.1, 48.0)
- added C31: 10uF, Capacitor_SMD:C_0805_2012Metric, F.Cu at (-129.1, 51.0)
- added C32: 10uF, Capacitor_SMD:C_0805_2012Metric, F.Cu at (-129.1, 54.0)
- added C33: 100nF, Capacitor_SMD:C_0805_2012Metric, F.Cu at (-129.1, 57.0)
- added C39: 10uF, Capacitor_SMD:C_1206_3216Metric, F.Cu at (-102.9, 124.3)
- added C4: 4.7uF, Capacitor_SMD:C_0805_2012Metric, B.Cu at (194.8, 74.3)
- added C40: 10uF, Capacitor_SMD:C_1206_3216Metric, F.Cu at (-141.7, 108.9)
- added C41: 10uF, Capacitor_SMD:C_1206_3216Metric, F.Cu at (-141.7, 112.2)
- added C42: 10uF, Capacitor_SMD:C_1206_3216Metric, F.Cu at (-102.9, 127.6)
- added C43: 1uF, Capacitor_SMD:C_0805_2012Metric, F.Cu at (-148.0, 99.7)
- added C44: 100nF, Capacitor_SMD:C_0805_2012Metric, F.Cu at (-148.0, 102.7)
- added C45: 10uF, Capacitor_SMD:C_1206_3216Metric, F.Cu at (-155.0, 97.4)
- added C46: 10uF, Capacitor_SMD:C_1206_3216Metric, F.Cu at (-141.7, 115.6)
- added C47: 100nF, Capacitor_SMD:C_0805_2012Metric, F.Cu at (-121.3, 152.9)
- added C48: 100nF, Capacitor_SMD:C_0805_2012Metric, F.Cu at (-121.3, 155.9)
- added C49: 100nF, Capacitor_SMD:C_0805_2012Metric, F.Cu at (-121.3, 158.9)
- added C5: 100nF, Capacitor_SMD:C_0805_2012Metric, B.Cu at (194.8, 77.3)
- added C50: 22uF, Capacitor_SMD:C_0805_2012Metric, F.Cu at (-148.0, 105.7)
- added C51: 10uF, Capacitor_SMD:C_1206_3216Metric, F.Cu at (-141.7, 118.9)
- added C52: 10uF, Capacitor_SMD:C_1206_3216Metric, F.Cu at (-136.1, 108.9)
- added C53: 1uF, Capacitor_SMD:C_0805_2012Metric, F.Cu at (-143.5, 90.7)
- added C54: 100nF, Capacitor_SMD:C_0805_2012Metric, F.Cu at (-143.5, 93.7)
- added C55: 10uF, Capacitor_SMD:C_1206_3216Metric, B.Cu at (178.5, 78.2)
- added C56: 1uF, Capacitor_SMD:C_0805_2012Metric, F.Cu at (-143.5, 96.7)
- added C57: 1uF, Capacitor_SMD:C_0805_2012Metric, F.Cu at (-143.5, 99.7)
- added C58: 10uF, Capacitor_SMD:C_1206_3216Metric, F.Cu at (-89.0, 167.8)
- added C59: 100nF, Capacitor_SMD:C_0805_2012Metric, F.Cu at (-121.3, 161.9)
- added C6: 47nF, Capacitor_SMD:C_0805_2012Metric, B.Cu at (194.8, 80.3)
- added C60: 100nF, Capacitor_SMD:C_0805_2012Metric, F.Cu at (-121.3, 165.0)
- added C61: 100nF, Capacitor_SMD:C_0805_2012Metric, F.Cu at (-121.3, 168.0)
- added C62: 470pF, Capacitor_SMD:C_0805_2012Metric, F.Cu at (-121.3, 171.0)
- added C63: 1uF, Capacitor_SMD:C_0805_2012Metric, F.Cu at (-121.3, 174.0)
- added C64: 22uF, Capacitor_SMD:C_0805_2012Metric, F.Cu at (-162.2, 107.1)
- added C65: 100nF, Capacitor_SMD:C_0805_2012Metric, F.Cu at (-162.2, 110.1)
- added C66: 100nF, Capacitor_SMD:C_0805_2012Metric, F.Cu at (-162.2, 113.2)
- added C67: 1uF, Capacitor_SMD:C_0805_2012Metric, F.Cu at (-162.2, 116.2)
- added C68: 100nF, Capacitor_SMD:C_0805_2012Metric, F.Cu at (-162.2, 119.2)
- added C69: 10uF, Capacitor_SMD:C_1206_3216Metric, F.Cu at (-136.1, 112.2)
- added C7: 10uF, Capacitor_SMD:C_1206_3216Metric, B.Cu at (57.5, 118.5)
- added C70: 100nF, Capacitor_SMD:C_0805_2012Metric, F.Cu at (-129.1, 60.1)
- added C71: 1uF, Capacitor_SMD:C_0805_2012Metric, F.Cu at (-143.5, 102.7)
- added C72: 100nF, Capacitor_SMD:C_0805_2012Metric, F.Cu at (-129.1, 63.1)
- added C73: 100nF, Capacitor_SMD:C_0805_2012Metric, F.Cu at (-124.6, 45.0)
- added C74: 100nF, Capacitor_SMD:C_0805_2012Metric, F.Cu at (-124.6, 48.0)
- added C75: 100nF, Capacitor_SMD:C_0805_2012Metric, F.Cu at (-124.6, 51.0)
- added C76: 100nF, Capacitor_SMD:C_0805_2012Metric, F.Cu at (-124.6, 54.0)
- added C77: 100nF, Capacitor_SMD:C_0805_2012Metric, F.Cu at (-124.6, 57.0)
- added C78: 100nF, Capacitor_SMD:C_0805_2012Metric, F.Cu at (-124.6, 60.1)
- added C79: 100nF, Capacitor_SMD:C_0805_2012Metric, F.Cu at (-124.6, 63.1)
- added C8: 10uF, Capacitor_SMD:C_1206_3216Metric, B.Cu at (55.0, 118.5)
- added C80: 100nF, Capacitor_SMD:C_0805_2012Metric, F.Cu at (-120.2, 45.0)
- added C81: 150pF, Capacitor_SMD:C_0805_2012Metric, F.Cu at (-120.2, 48.0)
- added C82: 5.6nF, Capacitor_SMD:C_0805_2012Metric, F.Cu at (-120.2, 51.0)
- added C83: 100nF, Capacitor_SMD:C_0805_2012Metric, F.Cu at (-143.5, 105.7)
- added C84: 10uF, Capacitor_SMD:C_0805_2012Metric, F.Cu at (-120.2, 54.0)
- added C85: 10uF, Capacitor_SMD:C_0805_2012Metric, F.Cu at (-120.2, 57.0)
- added C86: 100nF, Capacitor_SMD:C_0805_2012Metric, F.Cu at (-120.2, 60.1)
- added C87: 22uF, Capacitor_SMD:C_0805_2012Metric, F.Cu at (-139.1, 90.7)
- added C88: 100nF, Capacitor_SMD:C_0805_2012Metric, F.Cu at (-120.2, 63.1)
- added C9: 470nF, Capacitor_SMD:C_0805_2012Metric, B.Cu at (194.8, 83.3)
- added C97: 100nF, Capacitor_SMD:C_0805_2012Metric, F.Cu at (-101.4, 90.7)
- added C98: 100nF, Capacitor_SMD:C_0805_2012Metric, F.Cu at (-101.4, 93.7)
- added C99: 10uF, Capacitor_SMD:C_0805_2012Metric, F.Cu at (-101.4, 96.7)
- added D1: ESD5B5VL, Diode_SMD:D_SOD-523, B.Cu at (195.3, 98.3)
- added D2: ESD9B5.0ST5G, Diode_SMD:D_SOD-923, F.Cu at (-100.0, 110.1)
- added D3: LED, LED_SMD:LED_0805_2012Metric, F.Cu at (-127.9, 137.0)
- added FB1: BLM18BB600SN1, Inductor_SMD:L_0603_1608Metric, F.Cu at (-96.5, 173.7)
- added J1: RJ45_Abracon_ARJP11A-MASA-B-A-EMU2, Connector_RJ:RJ45_Abracon_ARJP11A-MA_Horizontal, F.Cu at (70.0, 96.3)
- added J2: USB_C_Receptacle_USB2.0_16P, Connector_USB:USB_C_Receptacle_HRO_TYPE-C-31-M-12, F.Cu at (54.0, 87.8)
- added J3: AFBR-1624Z, OptoDevice:Broadcom_AFBR-16xxZ_Horizontal, F.Cu at (95.1, 116.0)
- added J4: AFBR-2529Z, OptoDevice:Broadcom_AFBR-16xxZ_Horizontal, F.Cu at (82.6, 116.0)
- added J5: RF/COAXIAL SMA BHD JACK STR 50OHM SOLDER, Connector_Coaxial:SMA_Amphenol_132289_EdgeMount, F.Cu at (140.5, 89.8)
- added J6: SJ-3506-SMT-TR, MIKILAB_SJ_3506_SMT_TR:CUI_SJ-3506-SMT-TR, F.Cu at (132.5, 125.0)
- added J7: SJ-435107RS, MIKILAB_SJ_435107RS:CUI_SJ-435107RS, F.Cu at (138.4, 103.4)
- added J8: SJ-3506-SMT-TR, MIKILAB_SJ_3506_SMT_TR:CUI_SJ-3506-SMT-TR, F.Cu at (119.0, 125.0)
- added J9: SJ-3506-SMT-TR, MIKILAB_SJ_3506_SMT_TR:CUI_SJ-3506-SMT-TR, F.Cu at (105.0, 124.8)
- added J_BAT1: Conn_01x02, Connector_PinHeader_2.54mm:PinHeader_1x02_P2.54mm_Horizontal, B.Cu at (173.3, 128.4)
- added J_POW_BTN1: Conn_01x02, Connector_PinHeader_2.54mm:PinHeader_1x02_P2.54mm_Horizontal, B.Cu at (189.8, 126.4)
- added L1: 1uH, Inductor_SMD:L_Murata_DFE201610P, B.Cu at (195.3, 95.5)
- added L10: ferrite bead, Inductor_SMD:L_0603_1608Metric, F.Cu at (-141.5, 83.2)
- added L13: 18nH, Inductor_SMD:L_0603_1608Metric, F.Cu at (-103.5, 107.6)
- added L14: 120nH, Inductor_SMD:L_0603_1608Metric, F.Cu at (-103.5, 110.1)
- added L15: 22nH, Inductor_SMD:L_0603_1608Metric, F.Cu at (-103.5, 112.7)
- added L16: 36nH, Inductor_SMD:L_0603_1608Metric, F.Cu at (-103.5, 115.2)
- added L17: 100nH, Inductor_SMD:L_0603_1608Metric, F.Cu at (-103.5, 117.7)
- added L18: ferrite bead, Inductor_SMD:L_0805_2012Metric, F.Cu at (-130.1, 104.3)
- added L2: 1uH, Inductor_SMD:L_Coilcraft_XxL4020, B.Cu at (61.5, 122.5)
- added L21: ferrite bead, Inductor_SMD:L_0805_2012Metric, F.Cu at (-97.8, 124.0)
- added L22: ferrite bead, Inductor_SMD:L_0805_2012Metric, F.Cu at (-97.8, 126.7)
- added L23: ferrite bead, Inductor_SMD:L_0805_2012Metric, F.Cu at (-97.8, 129.5)
- added L24: ferrite bead, Inductor_SMD:L_0805_2012Metric, F.Cu at (-97.8, 132.2)
- added L3: ferrite bead, Inductor_SMD:L_0805_2012Metric, F.Cu at (-130.1, 90.5)
- added L4: ferrite bead, Inductor_SMD:L_0805_2012Metric, F.Cu at (-130.1, 93.3)
- added L5: ferrite bead, Inductor_SMD:L_0603_1608Metric, F.Cu at (-141.5, 80.7)
- added L6: ferrite bead, Inductor_SMD:L_0805_2012Metric, F.Cu at (-130.1, 96.0)
- added L8: ferrite bead, Inductor_SMD:L_0805_2012Metric, F.Cu at (-130.1, 98.8)
- added L9: ferrite bead, Inductor_SMD:L_0805_2012Metric, F.Cu at (-130.1, 101.5)
- added R1: 10K, Resistor_SMD:R_0805_2012Metric, B.Cu at (177.1, 88.0)
- added R10: 10K, Resistor_SMD:R_0805_2012Metric, B.Cu at (172.7, 96.8)
- added R11: 10K, Resistor_SMD:R_0805_2012Metric, B.Cu at (168.2, 88.0)
- added R12: 1M, Resistor_SMD:R_0805_2012Metric, B.Cu at (72.0, 114.5)
- added R13: 180K, Resistor_SMD:R_0805_2012Metric, B.Cu at (69.5, 114.6)
- added R15: 100m, Resistor_SMD:R_1206_3216Metric, B.Cu at (172.9, 80.6)
- added R16: 100m, Resistor_SMD:R_1206_3216Metric, B.Cu at (172.9, 83.9)
- added R18: 1k, Resistor_SMD:R_0805_2012Metric, F.Cu at (-127.9, 124.1)
- added R19: 1k, Resistor_SMD:R_0805_2012Metric, F.Cu at (-127.9, 127.0)
- added R2: 330, Resistor_SMD:R_0805_2012Metric, F.Cu at (-96.3, 152.9)
- added R23: 10K, Resistor_SMD:R_0805_2012Metric, F.Cu at (-112.4, 45.0)
- added R24: 10K, Resistor_SMD:R_0805_2012Metric, F.Cu at (-112.4, 47.9)
- added R25: 49.9, Resistor_SMD:R_0805_2012Metric, F.Cu at (-96.3, 155.8)
- added R3: 10K, Resistor_SMD:R_0805_2012Metric, B.Cu at (177.1, 91.0)
- added R30: 330, Resistor_SMD:R_0805_2012Metric, F.Cu at (-96.3, 158.8)
- added R33: 10K, Resistor_SMD:R_0805_2012Metric, F.Cu at (-112.4, 50.9)
- added R34: 12.1K, Resistor_SMD:R_0805_2012Metric, F.Cu at (-96.3, 161.7)
- added R35: 4.7K, Resistor_SMD:R_0805_2012Metric, F.Cu at (-96.3, 164.7)
- added R36: 4.7K, Resistor_SMD:R_0805_2012Metric, F.Cu at (-157.8, 107.1)
- added R37: 10K, Resistor_SMD:R_0805_2012Metric, F.Cu at (-91.9, 152.9)
- added R38: 10K, Resistor_SMD:R_0805_2012Metric, F.Cu at (-91.9, 155.8)
- added R39: 10K, Resistor_SMD:R_0805_2012Metric, F.Cu at (-91.9, 158.8)
- added R4: 187, Resistor_SMD:R_0805_2012Metric, B.Cu at (177.1, 93.9)
- added R40: 10K, Resistor_SMD:R_0805_2012Metric, F.Cu at (-91.9, 161.7)
- added R41: 5.1K, Resistor_SMD:R_0805_2012Metric, F.Cu at (-100.7, 69.5)
- added R42: 5.1K, Resistor_SMD:R_0805_2012Metric, F.Cu at (-100.7, 72.4)
- added R43: 10K, Resistor_SMD:R_0805_2012Metric, F.Cu at (-157.8, 110.1)
- added R44: 4.7K, Resistor_SMD:R_0805_2012Metric, F.Cu at (-157.8, 113.0)
- added R45: 4.7K, Resistor_SMD:R_0805_2012Metric, F.Cu at (-157.8, 116.0)
- added R46: 4.3K, Resistor_SMD:R_0805_2012Metric, F.Cu at (-135.9, 71.5)
- added R47: 10K, Resistor_SMD:R_0805_2012Metric, F.Cu at (-135.9, 74.4)
- added R48: 10K, Resistor_SMD:R_0805_2012Metric, F.Cu at (-135.9, 77.4)
- added R49: 10K, Resistor_SMD:R_0805_2012Metric, F.Cu at (-112.4, 53.8)
- added R5: 10K, Resistor_SMD:R_0805_2012Metric, B.Cu at (177.1, 96.8)
- added R50: 10K, Resistor_SMD:R_0805_2012Metric, F.Cu at (-112.4, 56.8)
- added R51: 100, Resistor_SMD:R_0805_2012Metric, F.Cu at (-135.9, 80.3)
- added R52: 4.7K, Resistor_SMD:R_0805_2012Metric, F.Cu at (-135.9, 83.3)
- added R53: 10K, Resistor_SMD:R_0805_2012Metric, F.Cu at (-112.4, 59.7)
- added R54: 1K, Resistor_SMD:R_0805_2012Metric, F.Cu at (-127.1, 108.7)
- added R55: 1K, Resistor_SMD:R_0805_2012Metric, F.Cu at (-127.1, 111.6)
- added R56: 10K, Resistor_SMD:R_0805_2012Metric, F.Cu at (-108.0, 45.0)
- added R58: 10K, Resistor_SMD:R_0805_2012Metric, F.Cu at (-138.4, 167.2)
- added R59: 10K, Resistor_SMD:R_0805_2012Metric, F.Cu at (-138.4, 170.1)
- added R6: 10K, Resistor_SMD:R_0805_2012Metric, B.Cu at (172.7, 88.0)
- added R68: 10K, Resistor_SMD:R_0805_2012Metric, F.Cu at (-108.0, 47.9)
- added R69: 10K, Resistor_SMD:R_0805_2012Metric, F.Cu at (-108.0, 50.9)
- added R7: 10K, Resistor_SMD:R_0805_2012Metric, B.Cu at (172.7, 91.0)
- added R70: 10K, Resistor_SMD:R_0805_2012Metric, F.Cu at (-108.0, 53.8)
- added R71: 10K, Resistor_SMD:R_0805_2012Metric, F.Cu at (-108.0, 56.8)
- added R73: 2.2K, Resistor_SMD:R_0805_2012Metric, F.Cu at (-163.9, 57.0)
- added R74: 2.2K, Resistor_SMD:R_0805_2012Metric, F.Cu at (-163.9, 60.0)
- added R75: 10K, Resistor_SMD:R_0805_2012Metric, F.Cu at (-157.8, 118.9)
- added R76: 10K, Resistor_SMD:R_0805_2012Metric, F.Cu at (-157.8, 121.9)
- added R77: 49.9, Resistor_SMD:R_0805_2012Metric, F.Cu at (-91.9, 164.7)
- added R78: 49.9, Resistor_SMD:R_0805_2012Metric, F.Cu at (-87.5, 152.9)
- added R79: 49.9, Resistor_SMD:R_0805_2012Metric, F.Cu at (-87.5, 155.8)
- added R8: 100, Resistor_SMD:R_0805_2012Metric, B.Cu at (172.7, 93.9)
- added R80: 33, Resistor_SMD:R_0805_2012Metric, F.Cu at (-87.5, 158.8)
- added R81: 33, Resistor_SMD:R_0805_2012Metric, F.Cu at (-87.5, 161.7)
- added R82: 10K, Resistor_SMD:R_0805_2012Metric, F.Cu at (-108.0, 59.7)
- added R83: 10K, Resistor_SMD:R_0805_2012Metric, F.Cu at (-103.6, 45.0)
- added R84: 10K, Resistor_SMD:R_0805_2012Metric, F.Cu at (-103.6, 47.9)
- added R85: 10K, Resistor_SMD:R_0805_2012Metric, F.Cu at (-103.6, 50.9)
- added R86: 10K, Resistor_SMD:R_0805_2012Metric, F.Cu at (-103.6, 53.8)
- added R87: 10K, Resistor_SMD:R_0805_2012Metric, F.Cu at (-103.6, 56.8)
- added R88: 10K, Resistor_SMD:R_0805_2012Metric, F.Cu at (-103.6, 59.7)
- added R89: 10K, Resistor_SMD:R_0805_2012Metric, F.Cu at (-99.2, 45.0)
- added R90: 10K, Resistor_SMD:R_0805_2012Metric, F.Cu at (-99.2, 47.9)
- added R91: 10K, Resistor_SMD:R_0805_2012Metric, F.Cu at (-99.2, 50.9)
- added R92: 10K, Resistor_SMD:R_0805_2012Metric, F.Cu at (-99.2, 53.8)
- added R93: 10K, Resistor_SMD:R_0805_2012Metric, F.Cu at (-99.2, 56.8)
- added R94: 10K, Resistor_SMD:R_0805_2012Metric, F.Cu at (-157.8, 124.8)
- added R95: 33, Resistor_SMD:R_0805_2012Metric, F.Cu at (-138.4, 173.1)
- added R96: 33, Resistor_SMD:R_0805_2012Metric, F.Cu at (-163.9, 62.9)
- added R97: 33, Resistor_SMD:R_0805_2012Metric, F.Cu at (-157.8, 127.8)
- added R98: 33, Resistor_SMD:R_0805_2012Metric, F.Cu at (-127.9, 130.0)
- added RESET1: TS3425UA-3x4x2.5-160, MIKILAB_TS3425UA_3x4x2_5_160:TS3425UA-3x4x2.5-160, F.Cu at (-161.2, 103.2)
- added RN10: 33, Resistor_SMD:R_Array_Concave_2x0603, F.Cu at (-140.2, 77.9)
- added RN2: 33, Resistor_SMD:R_Array_Concave_2x0603, F.Cu at (-148.5, 71.6)
- added RN3: 33, Resistor_SMD:R_Array_Concave_2x0603, F.Cu at (-148.5, 74.7)
- added RN4: 33, Resistor_SMD:R_Array_Concave_2x0603, F.Cu at (-148.5, 77.9)
- added RN5: 33, Resistor_SMD:R_Array_Concave_2x0603, F.Cu at (-144.3, 71.6)
- added RN6: 33, Resistor_SMD:R_Array_Concave_2x0603, F.Cu at (-144.3, 74.7)
- added RN7: 33, Resistor_SMD:R_Array_Concave_2x0603, F.Cu at (-144.3, 77.9)
- added RN8: 33, Resistor_SMD:R_Array_Concave_2x0603, F.Cu at (-140.2, 71.6)
- added RN9: 33, Resistor_SMD:R_Array_Concave_2x0603, F.Cu at (-140.2, 74.7)
- added U1: BQ25896, MIKILAB_ipc_qfn:IPC_QFN25P50_400X400X80L40X24T270N, B.Cu at (82.7, 100.2)
- added U10: W25Q128JVS, Package_SO:SOIC-8_5.3x5.3mm_P1.27mm, F.Cu at (-182.8, 124.2)
- added U11: ESP32-S31-WROOM-3, MIKILAB_ESP32_S31_WROOM_3:ESP32-S31-WROOM-3, F.Cu at (72.8, 68.8)
- added U12: Si4684-A10-GM, Package_DFN_QFN:QFN-48-1EP_7x7mm_P0.5mm_EP5.3x5.3mm, F.Cu at (-145.2, 170.3)
- added U13: TPD2E007DCKR, MIKILAB_TPD2E007DCKR:SOT65P210X110-3N, F.Cu at (-97.1, 90.8)
- added U14: TPD2E007DCKR, MIKILAB_TPD2E007DCKR:SOT65P210X110-3N, F.Cu at (-168.2, 60.5)
- added U15: ADG936BRUZ, MIKILAB_ADG936BRUZ:SOP65P640X120-20N, F.Cu at (-97.4, 105.2)
- added U17: 24AA025E64, Package_SO:SOIC-8_3.9x4.9mm_P1.27mm, F.Cu at (-160.2, 92.5)
- added U18: ADAU1467WBCPZ300R, MIKILAB_ADAU1467WBCPZ300RL:ADAU1467WBCPZ300, F.Cu at (-123.7, 71.6)
- added U19: LAN8720A, Package_DFN_QFN:VQFN-24-1EP_4x4mm_P0.5mm_EP2.5x2.5mm_ThermalVias, F.Cu at (-95.0, 169.3)
- added U2: BQ27441DRZR-G1B, Package_SON:Texas_S-PDSO-N12, B.Cu at (82.5, 90.0)
- added U20: TPS22994RUKT, MIKILAB_TPS22994RUKT:IC_TPS22994RUKT, F.Cu at (-130.1, 116.9)
- added U21: TPS22919DCK, Package_TO_SOT_SMD:SOT-363_SC-70-6, F.Cu at (-131.3, 109.0)
- added U22: TPS22919DCK, Package_TO_SOT_SMD:SOT-363_SC-70-6, F.Cu at (-131.3, 112.6)
- added U23: TPS22994RUKT, MIKILAB_TPS22994RUKT:IC_TPS22994RUKT, F.Cu at (-120.3, 143.3)
- added U24: 25AA1024-I_SM, Package_SO:SOIC-8_5.3x5.3mm_P1.27mm, F.Cu at (-126.1, 82.2)
- added U25: SN74AXC1T45DBVR, MIKILAB_SN74AXC1T45DBVR:SOT95P280X145-6N, F.Cu at (-96.0, 97.9)
- added U26: TPD2E007DCKR, MIKILAB_TPD2E007DCKR:SOT65P210X110-3N, F.Cu at (-168.2, 63.8)
- added U27: W25Q16JW, Package_SO:SOIC-8_5.3x5.3mm_P1.27mm, F.Cu at (-131.0, 169.2)
- added U28: TPD2E007DCKR, MIKILAB_TPD2E007DCKR:SOT65P210X110-3N, F.Cu at (-97.1, 94.1)
- added U29: TS5A23157DGS, Package_SO:TSSOP-10_3x3mm_P0.5mm, F.Cu at (-158.0, 57.8)
- added U3: TPS63020DSJT, MIKILAB_IC_TPS63020DSJT:IC_TPS63020DSJT, B.Cu at (61.4, 116.0)
- added U31: TMP117NAIDRVR, Package_SON:WSON-6-1EP_2x2mm_P0.65mm_EP1x1.6mm, F.Cu at (-98.2, 135.5)
- added U32: TMP117NAIDRVR, Package_SON:WSON-6-1EP_2x2mm_P0.65mm_EP1x1.6mm, F.Cu at (-98.2, 139.1)
- added U33: TMP117NAIDRVR, Package_SON:WSON-6-1EP_2x2mm_P0.65mm_EP1x1.6mm, F.Cu at (-98.2, 142.8)
- added U34: MCP23S17-E/ML, Package_DFN_QFN:QFN-28-1EP_6x6mm_P0.65mm_EP4.25x4.25mm, F.Cu at (-92.5, 47.6)
- added U35: 74HC138PW,118, Package_SO:TSSOP-16_4.4x5mm_P0.65mm, F.Cu at (-172.9, 124.0)
- added U36: MCP23S17-E/ML, Package_DFN_QFN:QFN-28-1EP_6x6mm_P0.65mm_EP4.25x4.25mm, F.Cu at (-92.5, 55.9)
- added U37: TMP117NAIDRVR, Package_SON:WSON-6-1EP_2x2mm_P0.65mm_EP1x1.6mm, F.Cu at (-98.2, 146.4)
- added U38: FSC-BT1058, MIKILAB_FSC_BT1058:FSC-BT1058, F.Cu at (127.0, 63.5)
- added U39: SRV05-4, Package_TO_SOT_SMD:SOT-23-6, F.Cu at (-112.0, 80.9)
- added U4: INA228, Package_SO:TSSOP-10_3x3mm_P0.5mm, B.Cu at (172.0, 72.1)
- added U40: SC16IS740IPW,128, Package_SO:TSSOP-16_4.4x5mm_P0.65mm, F.Cu at (-129.8, 144.0)
- added U5: XTAC5212IRGER, MIKILAB_XTAC5212IRGER:VQFN24_RGE_CORNERPADS_TEX, F.Cu at (-167.2, 68.7)
- added U6: TPS7A2012PDQN, Package_SON:Texas_X2SON-4_1x1mm_P0.65mm, B.Cu at (54.7, 113.1)
- added U7: TPS7A2018PDQN, Package_SON:Texas_X2SON-4_1x1mm_P0.65mm, B.Cu at (77.7, 109.6)
- added U8: INA228, Package_SO:TSSOP-10_3x3mm_P0.5mm, B.Cu at (172.0, 76.7)
- added U9: TPD2E007DCKR, MIKILAB_TPD2E007DCKR:SOT65P210X110-3N, F.Cu at (-168.2, 57.2)
- added X1: ASE-50.000MHZ-LC-T, Oscillator:Oscillator_SMD_Abracon_ASE-4Pin_3.2x2.5mm, F.Cu at (-89.2, 171.8)
- added Y1: ABM3B-12.288MHZ-10-1-U-T, Crystal:Crystal_SMD_5032-4Pin_5.0x3.2mm, F.Cu at (-147.0, 82.1)
- added Y2: ABM8-19.200MHZ-10-1-U-T, Crystal:Crystal_SMD_Abracon_ABM8AIG-4Pin_3.2x2.5mm, F.Cu at (-129.8, 155.9)
- added Y4: 12,288 MHz, Crystal:Crystal_SMD_2520-4Pin_2.5x2.0mm, F.Cu at (-127.9, 133.5)
Other:
- outline, holes or cut-outs redrawn
- copper layers 2 -> 6

Commit message: Power placemente (bottom layer) ... in progress
Parts:
- removed R1, R3: 10K, Resistor_SMD:R_0805_2012Metric
- added R20: 1k, Resistor_SMD:R_0805_2012Metric, B.Cu at (51.3, 62.8)
- J_POW_BTN1: footprint Connector_PinHeader_2.54mm:PinHeader_1x02_P2.54mm_Horizontal -> Connector_PinHeader_2.54mm:PinHeader_1x02_P2.54mm_Vertical
- R11: value 10K -> 10m; footprint Resistor_SMD:R_0805_2012Metric -> Resistor_SMD:R_1206_3216Metric_Pad1.30x1.75mm_HandSolder
- moved C9 142.1 mm to (54.8, 59.2)
- moved D1 140.6 mm to (56.5, 121.0)
- moved J_POW_BTN1 136.6 mm to (53.5, 118.0), turned to -90 degrees
- moved C10 132.6 mm to (59.0, 63.5), turned to -90 degrees
- moved J_BAT1 131.0 mm to (55.5, 71.0), turned to -90 degrees
- moved R10 125.1 mm to (51.3, 66.2), turned to 90 degrees
- moved C5 120.7 mm to (76.1, 98.7)
- moved R11 113.6 mm to (56.5, 68.0), turned to 0 degrees
- moved L1 112.2 mm to (83.1, 97.2)
- moved C6 110.0 mm to (86.1, 96.7), turned to 90 degrees
- moved C4 108.6 mm to (88.6, 96.7), turned to 90 degrees
- moved C3 106.9 mm to (91.1, 96.7), turned to 90 degrees
- moved C1 102.3 mm to (92.1, 101.7), turned to 90 degrees
- moved C55 100.9 mm to (81.1, 104.2)
- moved C2 98.2 mm to (94.1, 96.7), turned to 90 degrees
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Connections:
- R11 pad 1: GND -> /POWER/BAT+
- R11 pad 2: Net-(U2-BIN) -> /POWER/BQ25896_BAT
