File: hardware/kicad/HubAudio/POWER.kicad_sch (KiCad schematic)
At the start: 50 parts, among them U1 BQ25896, U2 BQ27441DRZR-G1B, U3 TPS63020DSJT, U4 INA228, U6 TPS7A2012PDQN, U7 TPS7A2018PDQN, U8 INA228

Commit message: Finalize I2C and SPI control architecture
Parts:
- removed C14: 10uF, Capacitor_SMD:C_1206_3216Metric, symbol Device:C
- removed C15: 1uF, Capacitor_SMD:C_1206_3216Metric, symbol Device:C
- removed C16: 100nF, Capacitor_SMD:C_0805_2012Metric, symbol Device:C
- removed L3: BLM21PG121SN1D, Inductor_SMD:L_0805_2012Metric, symbol Device:L
- added C118, C23: 47uF, Capacitor_SMD:C_1206_3216Metric, symbol Device:C
- added C55: 10uF, Capacitor_SMD:C_1206_3216Metric, symbol Device:C
- C1, C2, C7, C8: PNM (none) -> GRM31CR71E106KA12L
- C10, C17, C18, C19, C20: PNM (none) -> 12063C105KAT2A
- C11, C21, C22, C3, C5: PNM (none) -> GRM21BR71H104KA01L
- C12, C13: PNM (none) -> GRM31CR61E226ME15L
- C4: PNM (none) -> GRM21BR71C475KA73L
- C6: PNM (none) -> GRM21BR71H473KA01L
- C9: PNM (none) -> GRM21BR71H474KA88L
- D1: PNM (none) -> ESD5B5VL
- L1: value MHT201610SG-1R0M -> 1uH; PNM (none) -> DFE201612E-1R0M=P2
- L2: value XFL4020-102MEC -> 1uH; PNM (none) -> XFL4020-102MEC
- R1, R10, R11, R3, R5, R6, R7: PNM (none) -> RC0805FR-0710KL
- R12, R14: PNM (none) -> RC0805FR-071ML
- R13: PNM (none) -> RC0805FR-07180KL
- R15, R16: PNM (none) -> WSL1206R1000FEA
- R4: PNM (none) -> RC0805FR-07187RL
- R8: PNM (none) -> RC0805FR-07100RL
- R9: PNM (none) -> WSL1206R0100FEA
- U1: PNM (none) -> BQ25896RTWR
- U2: PNM (none) -> BQ27441DRZR-G1B
- U3: PACKAGE VSON-14 Texas Instruments -> (none); PNM (none) -> TPS63020DSJT
- U4, U8: PNM (none) -> INA228AQDGSRQ1
- U6: PNM (none) -> TPS7A2012PDQN
- U7: PNM (none) -> TPS7A2018PDQN
Connections:
- net V_OUT is gone; now on net VOUT: C7.1, C8.1, L1.2, U1.15 (SYS), U1.16 (SYS), U3.10 (VIN_10), U3.11 (VIN_11)
- net 3V3_ANALOG: now also C17.1, C19.1, U6.3 (EN), U6.4 (IN), U7.3 (EN), U7.4 (IN), U8.8 (Vbus), C118.2
- net 3V3_ANALOG_IN: no longer C17.1, C19.1, U6.3 (EN), U6.4 (IN), U7.3 (EN), U7.4 (IN), U8.8 (Vbus)
- net 3V3_DIGITAL: now also R1.1, R10.2, R3.1, R7.2, U4.8 (Vbus), C23.2
- net 3V3_DIGITAL_IN: no longer U4.8 (Vbus)
- net BQ25896_BAT: now also C55.1
- net GND: now also U3.13 (PS/SYNC), C118.1, C23.1, C55.2
- net VOUT: now reaches C11.1, U3.1 (VINA), U3.12 (EN)
- net VOUT: no longer U3.13 (PS/SYNC)
- no-connect marks 0 -> 1
Other:
- moved on the sheet: C11, C12, C13, C17, C18, C19, C20, C21, C22, L2, R12, R13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

Commit message: Update PCB power placement
Parts:
- removed R14: 1M, Resistor_SMD:R_0805_2012Metric, symbol Device:R
Other:
- moved on the sheet: R13
Changed lines of the file:
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@@
 	)
 	(junction
-		(at 116.84 106.68)
-		(diameter 0)
-		(color 0 0 0 0)
-	)
-	(junction
-		(at 125.73 111.76)
-		(diameter 0)
-		(color 0 0 0 0)
-	)
-	(junction
 		(at 45.72 25.4)
 		(diameter 0)
@@
 	)
 	(junction
-		(at 125.73 99.06)
-		(diameter 0)
-		(color 0 0 0 0)
-	)
-	(junction
 		(at 170.18 45.72)
 		(diameter 0)
@@
 	)
 	(junction
+		(at 116.84 106.68)
+		(diameter 0)
+		(color 0 0 0 0)
+	)
+	(junction
 		(at 127 26.67)
 		(diameter 0)
@@
 	(wire
 		(pts
-			(xy 116.84 99.06) (xy 125.73 99.06)
-		)
-		(stroke
-			(width 0)
-			(type default)
-		)
-	)
-	(wire
-		(pts
 			(xy 67.31 175.26) (xy 72.39 175.26)
 		)
@@
 	(wire
 		(pts
-			(xy 125.73 111.76) (xy 132.08 111.76)
-		)
-		(stroke
-			(width 0)
-			(type default)
-		)
-	)
-	(wire
-		(pts
 			(xy 114.3 68.58) (xy 120.65 68.58)
 		)
@@
 	(wire
 		(pts
-			(xy 125.73 106.68) (xy 125.73 111.76)
-		)
-		(stroke
-			(width 0)
-			(type default)
-		)
-	)
-	(wire
-		(pts
 			(xy 64.77 99.06) (xy 69.85 99.06)
 		)
@@
 	(wire
 		(pts
-			(xy 125.73 99.06) (xy 132.08 99.06)
+			(xy 116.84 99.06) (xy 132.08 99.06)
 		)
 		(stroke
@@
 	(wire
 		(pts
-			(xy 105.41 111.76) (xy 125.73 111.76)
+			(xy 105.41 111.76) (xy 132.08 111.76)
 		)
 		(stroke
@@
 	(symbol
 		(lib_id "Device:R")
-		(at 125.73 102.87 180)
-		(unit 1)
-		(body_style 1)
-		(exclude_from_sim no)
-		(in_bom yes)
-		(on_board yes)
-		(in_pos_files yes)
-		(dnp no)
-		(property "Reference" "R14"
-			(at 123.698 103.124 90)
-			(show_name no)
-			(do_not_autoplace no)
-			(effects
-				(font
-					(size 1.27 1.27)
-				)
-			)
-		)
-		(property "Value" "1M"
-			(at 126.492 102.87 90)
-			(show_name no)
-			(do_not_autoplace no)
-			(effects
-				(font
-					(size 1.27 1.27)
-				)
-				(justify top)
-			)
-		)
-		(property "Footprint" "Resistor_SMD:R_0805_2012Metric"
-			(at 127.508 102.87 90)
-			(hide yes)
-			(show_name no)
-			(do_not_autoplace no)
-			(effects
-				(font
-					(size 1.27 1.27)
-				)
-			)
-		)
-		(property "Datasheet" ""
-			(at 125.73 102.87 0)
-			(hide yes)
-			(show_name no)
-			(do_not_autoplace no)
-			(effects
-				(font
-					(size 1.27 1.27)
-				)
-			)
-		)
-		(property "Description" "RC0805FR-071ML"
-			(at 125.73 102.87 0)
-			(hide yes)
-			(show_name no)
-			(do_not_autoplace no)
-			(effects
-				(font
-					(size 1.27 1.27)
-				)
-			)
-		)
-		(property "PNM" "RC0805FR-071ML"
-			(at 125.73 102.87 90)
-			(hide yes)
-			(show_name no)
-			(do_not_autoplace no)
-			(effects
-				(font
-					(size 1.27 1.27)
-				)
-			)
-		)
-		(pin "1"
-		)
-		(pin "2"
-		)
-		(instances
-			(project "HubAudio"
-				(path "/841d8022-3a94-443e-97aa-a99a12889684/be5acd16-8a33-4b43-9869-78b6acaaceab"
-					(reference "R14")
-					(unit 1)
-				)
-			)
-		)
-	)
-	(symbol
-		(lib_id "Device:R")
 		(at 95.25 72.39 180)
 		(unit 1)
@@
 	(symbol
 		(lib_id "Device:R")
-		(at 116.84 110.49 180)
+		(at 120.65 106.68 270)
 		(unit 1)
 		(body_style 1)
@@
 		(dnp no)
 		(property "Reference" "R13"
-			(at 114.808 110.744 90)
+			(at 120.904 108.712 90)
 			(show_name no)
 			(do_not_autoplace no)
@@
 		)
 		(property "Value" "180K"
-			(at 117.602 110.49 90)
+			(at 120.65 105.918 90)
 			(show_name no)
 			(do_not_autoplace no)
@@
 		)
 		(property "Footprint" "Resistor_SMD:R_0805_2012Metric"
-			(at 118.618 110.49 90)
+			(at 120.65 104.902 90)
 			(hide yes)
 			(show_name no)
@@
 		)
 		(property "Datasheet" ""
-			(at 116.84 110.49 0)
+			(at 120.65 106.68 0)
 			(hide yes)
 			(show_name no)
@@
 		)
 		(property "Description" "RC0805FR-07180KL"
-			(at 116.84 110.49 0)
+			(at 120.65 106.68 0)
 			(hide yes)
 			(show_name no)
@@
 		)
 		(property "PNM" "RC0805FR-07180KL"
-			(at 116.84 110.49 90)
+			(at 120.65 106.68 90)
 			(hide yes)
 			(show_name no)
@@
 	(symbol
 		(lib_id "power:GND")
-		(at 116.84 114.3 0)
+		(at 124.46 106.68 90)
 		(unit 1)
 		(body_style 1)
@@
 		(dnp no)
 		(property "Reference" "#PWR019"
-			(at 116.84 120.65 0)
+			(at 130.81 106.68 0)
 			(hide yes)
 			(show_name no)
@@
 		)
 		(property "Value" "GND"
-			(at 119.634 117.348 0)
+			(at 128.27 106.68 0)
 			(show_name no)
 			(do_not_autoplace no)
@@
 		)
 		(property "Footprint" ""
-			(at 116.84 114.3 0)
+			(at 124.46 106.68 0)
 			(hide yes)
 			(show_name no)
@@
 		)
 		(property "Datasheet" ""
-			(at 116.84 114.3 0)
+			(at 124.46 106.68 0)
 			(hide yes)
 			(show_name no)
@@
 		)
 		(property "Description" "Power symbol creates a global label with name \"GND\" , ground"
-			(at 116.84 114.3 0)
+			(at 124.46 106.68 0)
 			(hide yes)
 			(show_name no)

Commit message: Power placemente (bottom layer) ... in progress
Parts:
- removed R1, R3: 10K, Resistor_SMD:R_0805_2012Metric, symbol Device:R
- removed R9: 10m, Resistor_SMD:R_1206_3216Metric, symbol Device:R
- added R20: 1k, Resistor_SMD:R_0805_2012Metric, symbol Device:R
- J_POW_BTN1: footprint Connector_PinHeader_2.54mm:PinHeader_1x02_P2.54mm_Horizontal -> Connector_PinHeader_2.54mm:PinHeader_1x02_P2.54mm_Vertical
- R11: value 10K -> 10m; footprint Resistor_SMD:R_0805_2012Metric -> Resistor_SMD:R_1206_3216Metric_Pad1.30x1.75mm_HandSolder; PNM RC0805FR-0710KL -> ERJ-8CWFR010V
Connections:
- net BAT+: now also R11.1
- net BQ25896_BAT: now also R11.2
- net GND: now also R20.2; no longer R11.1
- net at U2.10 (BIN): now also R20.1; no longer R11.2
